Commit message: YOLO Shared Memory mimarisine gecildi ve UI hatalari cözuldu

File: install/zed_wrapper/share/zed_wrapper/urdf/zed_descr.urdf.xacro (robot description, xacro)
@@ -1,30 +1 @@
-<?xml version="1.0"?>
-<!--
-// Copyright 2025 Stereolabs
-//
-// Licensed under the Apache License, Version 2.0 (the "License");
-// you may not use this file except in compliance with the License.
-// You may obtain a copy of the License at
-//
-//      http://www.apache.org/licenses/LICENSE-2.0
-//
-// Unless required by applicable law or agreed to in writing, software
-// distributed under the License is distributed on an "AS IS" BASIS,
-// WITHOUT WARRANTIES OR CONDITIONS OF ANY KIND, either express or implied.
-// See the License for the specific language governing permissions and
-// limitations under the License.
--->
-<robot name="stereolabs_camera" xmlns:xacro="http://ros.org/wiki/xacro">
-  <xacro:arg name="camera_name"   default="zed" />
-  <xacro:arg name="camera_model"  default="zed" />
-  <xacro:arg name="custom_baseline"  default="0.0" />
-  <!-- If GNSS fusion is enabled the position of the antenna with respect to the camera mount point is required -->
-  <xacro:arg name="enable_gnss"   default="false" />
-  <xacro:arg name="gnss_x" default="0.0" />
-  <xacro:arg name="gnss_y" default="0.0" />
-  <xacro:arg name="gnss_z" default="0.0" />
-  <xacro:include filename="$(find zed_wrapper)/urdf/zed_macro.urdf.xacro" />
-  <xacro:zed_camera name="$(arg camera_name)" model="$(arg camera_model)" custom_baseline="$(arg custom_baseline)" enable_gnss="$(arg enable_gnss)">
-	    <origin xyz="$(arg gnss_x) $(arg gnss_y) $(arg gnss_z)" rpy="0 0 0"/>
-  </xacro:zed_camera>
-</robot>
+/home/baris/mavivatan_ws/src/zed-ros2-wrapper/zed_wrapper/urdf/zed_descr.urdf.xacro

File: install/zed_wrapper/share/zed_wrapper/urdf/zed_macro.urdf.xacro (robot description, xacro)
@@ -1,298 +1 @@
-<?xml version="1.0"?>
-<!--
-// Copyright 2025 Stereolabs
-//
-// Licensed under the Apache License, Version 2.0 (the "License");
-// you may not use this file except in compliance with the License.
-// You may obtain a copy of the License at
-//
-//      http://www.apache.org/licenses/LICENSE-2.0
-//
-// Unless required by applicable law or agreed to in writing, software
-// distributed under the License is distributed on an "AS IS" BASIS,
-// WITHOUT WARRANTIES OR CONDITIONS OF ANY KIND, either express or implied.
-// See the License for the specific language governing permissions and
-// limitations under the License.
--->
-<robot xmlns:xacro="http://wiki.ros.org/xacro">
-  <xacro:property name="M_PI"     value="3.1415926535897931" />
-  <!--
-    Parameters:
-      - name: the camera's name.  should match the parameter sent to the launch file for this camera
-      - model: the type of camera, one of zed, zedm, zed2, zed2i, zedx, zedxm, virtual
-      - enable_gnss: if true enable the URDF link
-  -->
-  <xacro:macro name="zed_camera" params="name=zed model=zed enable_gnss=false custom_baseline=0 *gnss_origin">
-    <xacro:if value="${model == 'zed'}">
-      <xacro:property name="baseline" value="0.12" />
-      <xacro:property name="height" value="0.03" />
-      <xacro:property name="bottom_slope" value="0.05" />
-      <xacro:property name="screw_offset_x" value="0.0" />
-      <xacro:property name="screw_offset_z" value="0.0" />
-      <xacro:property name="optical_offset_x" value="-0.01" />
-      <xacro:property name="mono" value="false" />
-      <xacro:property name="mat" value="0.8 0.8 0.8 1.0" />
-    </xacro:if>
-    <xacro:if value="${model == 'zedm'}">
-      <xacro:property name="baseline" value="0.063" />
-      <xacro:property name="height" value="0.0265" />
-      <xacro:property name="bottom_slope" value="0.0" />
-      <xacro:property name="screw_offset_x" value="0.0" />
-      <xacro:property name="screw_offset_z" value="0.0" />
-      <xacro:property name="optical_offset_x" value="0.0" />
-      <xacro:property name="mono" value="false" />
-      <xacro:property name="mat" value="0 0 0 1.0" />
-    </xacro:if>
-    <xacro:if value="${model == 'zed2'}">
-      <xacro:property name="baseline" value="0.12" />
-      <xacro:property name="height" value="0.03" />
-      <xacro:property name="bottom_slope" value="0.05" />
-      <xacro:property name="screw_offset_x" value="0.0" />
-      <xacro:property name="screw_offset_z" value="0.0" />
-      <xacro:property name="optical_offset_x" value="-0.01" />
-      <xacro:property name="mono" value="false" />
-      <xacro:property name="mat" value="0.25 0.25 0.25 1.0" />
-    </xacro:if>
-    <xacro:if value="${model == 'zed2i'}">
-      <xacro:property name="baseline" value="0.12" />
-      <xacro:property name="height" value="0.03" />
-      <xacro:property name="bottom_slope" value="0.0" />
-      <xacro:property name="screw_offset_x" value="-0.01" />
-      <xacro:property name="screw_offset_z" value="0.0" />
-      <xacro:property name="optical_offset_x" value="-0.01" />
-      <xacro:property name="mono" value="false" />
-      <xacro:property name="mat" value="0.25 0.25 0.25 1.0" />
-    </xacro:if>
-    <xacro:if value="${model == 'zedx'}">
-      <xacro:property name="baseline" value="0.12" />
-      <xacro:property name="height" value="0.032" />
-      <xacro:property name="bottom_slope" value="0.0" />
-      <xacro:property name="screw_offset_x" value="0.0" />
-      <xacro:property name="screw_offset_z" value="-0.016" />
-      <xacro:property name="optical_offset_x" value="-0.01" />
-      <xacro:property name="mono" value="false" />
-      <xacro:property name="mat" value="0.25 0.25 0.25 1.0" />
-    </xacro:if>
-    <xacro:if value="${model == 'zedxhdr'}">
-      <xacro:property name="baseline" value="0.12" />
-      <xacro:property name="height" value="0.032" />
-      <xacro:property name="bottom_slope" value="0.0" />
-      <xacro:property name="screw_offset_x" value="0.0" />
-      <xacro:property name="screw_offset_z" value="-0.016" />
-      <xacro:property name="optical_offset_x" value="-0.01" />
-      <xacro:property name="mono" value="false" />
-      <xacro:property name="mat" value="0.25 0.25 0.25 1.0" />
-    </xacro:if>
-    <xacro:if value="${model == 'zedxm'}">
-      <xacro:property name="baseline" value="0.05" />
-      <xacro:property name="height" value="0.032" />
-      <xacro:property name="bottom_slope" value="0.0" />
-      <xacro:property name="screw_offset_x" value="0.0" />
-      <xacro:property name="screw_offset_z" value="-0.016" />
-      <xacro:property name="optical_offset_x" value="-0.01" />
-      <xacro:property name="mono" value="false" />
-      <xacro:property name="mat" value="0.25 0.25 0.25 1.0" />
-    </xacro:if>
-    <xacro:if value="${model == 'zedxhdrmini'}">
-      <xacro:property name="baseline" value="0.05" />
-      <xacro:property name="height" value="0.032" />
-      <xacro:property name="bottom_slope" value="0.0" />
-      <xacro:property name="screw_offset_x" value="0.0" />
-      <xacro:property name="screw_offset_z" value="-0.016" />
-      <xacro:property name="optical_offset_x" value="-0.01" />
-      <xacro:property name="mono" value="false" />
-      <xacro:property name="mat" value="0.25 0.25 0.25 1.0" />
-    </xacro:if>
-    <xacro:if value="${model == 'zedxhdrmax'}">
-      <xacro:property name="baseline" value="0.170" />
-      <xacro:property name="height" value="0.032" />
-      <xacro:property name="bottom_slope" value="0.0" />
-      <xacro:property name="screw_offset_x" value="0.0" />
-      <xacro:property name="screw_offset_z" value="-0.016" />
-      <xacro:property name="optical_offset_x" value="-0.01" />
-      <xacro:property name="mono" value="false" />
-      <xacro:property name="mat" value="0.25 0.25 0.25 1.0" />
-    </xacro:if>
-    <xacro:if value="${model == 'virtual'}">
-      <xacro:property name="baseline" value="${custom_baseline}" />
-      <xacro:property name="height" value="0.031" />
-      <xacro:property name="bottom_slope" value="0.0" />
-      <xacro:property name="screw_offset_x" value="0.00" />
-      <xacro:property name="screw_offset_z" value="-0.0155" />
-      <xacro:property name="optical_offset_x" value="0.0" />
-      <xacro:property name="mono" value="false" />
-      <xacro:property name="mat" value="0.25 0.25 0.25 1.0" />
-    </xacro:if>
-    <xacro:if value="${model == 'zedxonegs'}">
-      <xacro:property name="baseline" value="0.0" />
-      <xacro:property name="height" value="0.031" />
-      <xacro:property name="bottom_slope" value="0.0" />
-      <xacro:property name="screw_offset_x" value="0.0" />
-      <xacro:property name="screw_offset_z" value="-0.0155" />
-      <xacro:property name="optical_offset_x" value="0.0" />
-      <xacro:property name="mono" value="true" />
-      <xacro:property name="mat" value="0.25 0.25 0.25 1.0" />
-    </xacro:if>
-    <xacro:if value="${model == 'zedxone4k'}">
-      <xacro:property name="baseline" value="0.0" />
-      <xacro:property name="height" value="0.031" />
-      <xacro:property name="bottom_slope" value="0.0" />
-      <xacro:property name="screw_offset_x" value="0.00" />
-      <xacro:property name="screw_offset_z" value="-0.0155" />
-      <xacro:property name="optical_offset_x" value="0.0" />
-      <xacro:property name="mono" value="true" />
-      <xacro:property name="mat" value="0.25 0.25 0.25 1.0" />
-    </xacro:if>
-    <xacro:if value="${model == 'zedxonehdr'}">
-      <xacro:property name="baseline" value="0.0" />
-      <xacro:property name="height" value="0.025" />
-      <xacro:property name="bottom_slope" value="0.0" />
-      <xacro:property name="screw_offset_x" value="0.00" />
-      <xacro:property name="screw_offset_z" value="-0.0125" />
-      <xacro:property name="optical_offset_x" value="0.0" />
-      <xacro:property name="mono" value="true" />
-      <xacro:property name="mat" value="0.25 0.25 0.25 1.0" />
-    </xacro:if>
-    <!-- Camera mounting point (the threaded screw hole in the bottom) -->
-    <link name="${name}_camera_link" />
-    <!-- Camera Center -->
-    <link name="${name}_camera_center">
-      <xacro:unless value="${model == 'virtual'}">
-        <visual>
-          <origin xyz="${screw_offset_x} 0 ${screw_offset_z}" rpy="0 0 0"/>
-          <geometry>
-            <mesh filename="file://$(find zed_msgs)/meshes/${model}.stl"/>
-          </geometry>
-            <material name="zed_mat">
-              <color rgba="${mat}"/>
-            </material>
-        </visual>
-        <collision>
-          <origin xyz="${screw_offset_x} 0 ${screw_offset_z}" rpy="0 0 0"/>
-          <geometry>
-            <mesh filename="file://$(find zed_msgs)/meshes/${model}.stl"/>
-          </geometry>
-        </collision>
-      </xacro:unless>
-    </link>
-    <joint name="${name}_camera_center_joint" type="fixed">
-      <parent link="${name}_camera_link"/>
-      <child link="${name}_camera_center"/>
-      <origin xyz="0 0 ${height/2}" rpy="0 ${bottom_slope} 0" />
-    </joint>
-    <xacro:unless value="${mono}">
-      <!-- Left Camera -->
-      <link name="${name}_left_camera_frame">
-        <xacro:if value="${model == 'virtual'}">
-          <visual>
-            <origin xyz="0 0 0" rpy="0 0 0"/>
-            <geometry>
-              <mesh filename="file://$(find zed_msgs)/meshes/${model}.stl"/>
-            </geometry>
-            <material name="zed_mat">
-              <color rgba="${mat}"/>
-            </material>
-          </visual>
-          <collision>
-            <origin xyz="0 0 0" rpy="0 0 0"/>
-            <geometry>
-              <mesh filename="file://$(find zed_msgs)/meshes/${model}.stl"/>
-            </geometry>
-          </collision>
-        </xacro:if>
-      </link>
-      <joint name="${name}_left_camera_joint" type="fixed">
-        <parent link="${name}_camera_center"/>
-        <child link="${name}_left_camera_frame"/>
-        <origin xyz="${optical_offset_x} ${baseline/2} 0" rpy="0 0 0" />
-      </joint>
-      <link name="${name}_left_camera_frame_optical"/>
-      <joint name="${name}_left_camera_joint_optical" type="fixed">
-        <origin xyz="0 0 0" rpy="-${M_PI/2} 0.0 -${M_PI/2}"/>
-        <parent link="${name}_left_camera_frame"/>
-        <child link="${name}_left_camera_frame_optical"/>
-      </joint>
-      <!-- Right Camera -->
-      <link name="${name}_right_camera_frame">
-        <xacro:if value="${model == 'virtual'}">
-          <visual>
-            <origin xyz="0 0 0" rpy="0 0 0"/>
-            <geometry>
-              <mesh filename="file://$(find zed_msgs)/meshes/${model}.stl"/>
-            </geometry>
-            <material name="zed_mat">
-              <color rgba="${mat}"/>
-            </material>
-          </visual>
-          <collision>
-            <origin xyz="0 0 0" rpy="0 0 0"/>
-            <geometry>
-              <mesh filename="file://$(find zed_msgs)/meshes/${model}.stl"/>
-            </geometry>
-          </collision>
-        </xacro:if>
-      </link>
-      <joint name="${name}_right_camera_joint" type="fixed">
-        <parent link="${name}_camera_center"/>
-        <child link="${name}_right_camera_frame"/>
-        <origin xyz="${optical_offset_x} -${baseline/2} 0" rpy="0 0 0" />
-      </joint>
-      <link name="${name}_right_camera_frame_optical"/>
-      <joint name="${name}_right_camera_joint_optical" type="fixed">
-        <origin xyz="0 0 0" rpy="-${M_PI/2} 0.0 -${M_PI/2}"/>
-        <parent link="${name}_right_camera_frame"/>
-        <child link="${name}_right_camera_frame_optical"/>
-      </joint>
-      <!-- ZED2 Sensors -->
-      <xacro:if value="${model == 'zed2'}">
-        <link name="${name}_mag_link" />
-        <joint name="${name}_mag_joint" type="fixed">
-          <parent link="${name}_camera_center"/>
-          <child link="${name}_mag_link"/>
-          <origin xyz="0 0 0" rpy="0 0 0" />
-        </joint>
-        <link name="${name}_baro_link" />
-        <joint name="${name}_baro_joint" type="fixed">
-          <parent link="${name}_camera_center"/>
-          <child link="${name}_baro_link"/>
-          <origin xyz="0 0 0" rpy="0 0 0" />
-        </joint>
-        <link name="${name}_temp_left_link" />
-        <joint name="${name}_temp_left_joint" type="fixed">
-          <parent link="${name}_left_camera_frame"/>
-          <child link="${name}_temp_left_link"/>
-          <origin xyz="0 0 0" rpy="0 0 0" />
-        </joint>
-        <link name="${name}_temp_right_link" />
-        <joint name="${name}_temp_right_joint" type="fixed">
-          <parent link="${name}_right_camera_frame"/>
-          <child link="${name}_temp_right_link"/>
-          <origin xyz="0 0 0" rpy="0 0 0" />
-        </joint>
-      </xacro:if>
-    </xacro:unless>
-    <xacro:if value="${mono}">
-      <!-- Camera -->
-      <link name="${name}_camera_frame" />
-      <joint name="${name}_camera_joint" type="fixed">
-        <parent link="${name}_camera_center"/>
-        <child link="${name}_camera_frame"/>
-        <origin xyz="${optical_offset_x} 0 0" rpy="0 0 0" />
-      </joint>
-      <link name="${name}_camera_frame_optical"/>
-      <joint name="${name}_camera_optical_joint" type="fixed">
-        <origin xyz="0 0 0" rpy="-${M_PI/2} 0.0 -${M_PI/2}"/>
-        <parent link="${name}_camera_frame"/>
-        <child link="${name}_camera_frame_optical"/>
-      </joint>
-    </xacro:if>
-    <xacro:if value="${enable_gnss}">
-      <link name="${name}_gnss_link" />
-      <joint name="${name}_gnss_joint" type="fixed">
-        <parent link="${name}_camera_link"/>
-        <child link="${name}_gnss_link"/>
-        <xacro:insert_block name="gnss_origin" />
-      </joint>
-    </xacro:if>
-  </xacro:macro>
-</robot>
+/home/baris/mavivatan_ws/src/zed-ros2-wrapper/zed_wrapper/urdf/zed_macro.urdf.xacro
